File: Omniplex.kicad_pcb (KiCad board)
At the start: 4 copper layers, 116.2 x 82.6 mm, 89 parts, among them J1 Conn_Coaxial, J2 Conn_Coaxial, J3 Conn_Coaxial, J4 Conn_Coaxial, J5 Conn_Coaxial, J6 Conn_Coaxial, J7 Conn_Coaxial, J8 Conn_Coaxial, K1 TE_PCH-1xxx2M, K10 TE_PCH-1xxx2M, K11 TE_PCH-1xxx2M, K12 TE_PCH-1xxx2M, K13 TE_PCH-1xxx2M, K14 TE_PCH-1xxx2M, K15 TE_PCH-1xxx2M, K16 TE_PCH-1xxx2M, K2 TE_PCH-1xxx2M, K3 TE_PCH-1xxx2M, K4 TE_PCH-1xxx2M, K5 TE_PCH-1xxx2M, K6 TE_PCH-1xxx2M, K7 TE_PCH-1xxx2M, K8 TE_PCH-1xxx2M, K9 TE_PCH-1xxx2M, Q1 BS170F, Q10 BS170F, Q11 BS170F, Q12 BS170F, Q13 BS170F, Q14 BS170F, Q15 BS170F, Q16 BS170F, Q2 BS170F, Q3 BS170F, Q4 BS170F, Q5 BS170F, Q6 BS170F, Q7 BS170F, Q8 BS170F, Q9 BS170F

Commit message: asdf
Routing:
- net Net-(D13-Pad2): track 68.5 -> 66.6 mm
- net Net-(D15-Pad2): track 64.4 -> 62.7 mm
- net Net-(D3-Pad2): track 103.4 -> 101.8 mm
- net Net-(D5-Pad2): track 93.3 -> 92.5 mm
- net Net-(D9-Pad2): track 99.0 -> 98.4 mm
- net Net-(D10-Pad2): track 50.8 -> 50.3 mm

Commit message: asdf
Other:
- board text added: "Elchisoft"
- board text added: "Omniplex V1"
